Commit message: works with OpenDoorRL initial commit

File: urdf/bit_humanoid.urdf (robot description, URDF)
Before this commit: robot PatrolRobot, 29 links, 28 joints
Links:
- added link base_link
Joints:
- added joint torso: type fixed, parent base_link, child torso, origin xyz=0 0 0 rpy=0 0 0

Commit message: 1. corrected names in mesh references; 2. corrected floating base sensor placement

File: urdf/bit_humanoid.urdf (robot description, URDF)
Before this commit: robot bit_humanoid, 30 links, 29 joints
Links:
- link LArm0: geometry collision mesh filename=package://bit_humanoid/meshes/LArm0.STL; visual mesh filename=package://bit_humanoid/meshes/LArm0.STL
- link LArm1: geometry collision mesh filename=package://bit_humanoid/meshes/LArm1.STL; visual mesh filename=package://bit_humanoid/meshes/LArm1.STL
- link LArm2: geometry collision mesh filename=package://bit_humanoid/meshes/LArm2.STL; visual mesh filename=package://bit_humanoid/meshes/LArm2.STL
- link LArm3: geometry collision mesh filename=package://bit_humanoid/meshes/LArm3.STL; visual mesh filename=package://bit_humanoid/meshes/LArm3.STL
- link LArm4: geometry collision mesh filename=package://bit_humanoid/meshes/LArm4.STL; visual mesh filename=package://bit_humanoid/meshes/LArm4.STL
- link LArm5: geometry collision mesh filename=package://bit_humanoid/meshes/LArm5.STL; visual mesh filename=package://bit_humanoid/meshes/LArm5.STL
- link LArm6: geometry collision mesh filename=package://bit_humanoid/meshes/LArm6.STL; visual mesh filename=package://bit_humanoid/meshes/LArm6.STL
- link LArm7: geometry collision mesh filename=package://bit_humanoid/meshes/LArm7.STL; visual mesh filename=package://bit_humanoid/meshes/LArm7.STL
- link RArm0: geometry collision mesh filename=package://bit_humanoid/meshes/RArm0.STL; visual mesh filename=package://bit_humanoid/meshes/RArm0.STL
- link RArm1: geometry collision mesh filename=package://bit_humanoid/meshes/RArm1.STL; visual mesh filename=package://bit_humanoid/meshes/RArm1.STL
- link RArm2: geometry collision mesh filename=package://bit_humanoid/meshes/RArm2.STL; visual mesh filename=package://bit_humanoid/meshes/RArm2.STL
- link RArm3: geometry collision mesh filename=package://bit_humanoid/meshes/RArm3.STL; visual mesh filename=package://bit_humanoid/meshes/RArm3.STL
- link RArm4: geometry collision mesh filename=package://bit_humanoid/meshes/RArm4.STL; visual mesh filename=package://bit_humanoid/meshes/RArm4.STL
- link RArm5: geometry collision mesh filename=package://bit_humanoid/meshes/RArm5.STL; visual mesh filename=package://bit_humanoid/meshes/RArm5.STL
- link RArm6: geometry collision mesh filename=package://bit_humanoid/meshes/RArm6.STL; visual mesh filename=package://bit_humanoid/meshes/RArm6.STL
- link RArm7: geometry collision mesh filename=package://bit_humanoid/meshes/RArm7.STL; visual mesh filename=package://bit_humanoid/meshes/RArm7.STL
- link lanklepitch: geometry collision mesh filename=package://bit_humanoid/meshes/lanklepitch.STL; visual mesh filename=package://bit_humanoid/meshes/lanklepitch.STL
- link lankleroll: geometry collision mesh filename=package://bit_humanoid/meshes/lankleroll.STL; visual mesh filename=package://bit_humanoid/meshes/lankleroll.STL
- link lhippitch: geometry collision mesh filename=package://bit_humanoid/meshes/lhippitch.STL; visual mesh filename=package://bit_humanoid/meshes/lhippitch.STL
- link lhiproll: geometry collision mesh filename=package://bit_humanoid/meshes/lhiproll.STL; visual mesh filename=package://bit_humanoid/meshes/lhiproll.STL
- link lhipyaw: geometry collision mesh filename=package://bit_humanoid/meshes/lhipyaw.STL; visual mesh filename=package://bit_humanoid/meshes/lhipyaw.STL
- link lkneepitch: geometry collision mesh filename=package://bit_humanoid/meshes/lkneepitch.STL; visual mesh filename=package://bit_humanoid/meshes/lkneepitch.STL
- link ranklepitch: geometry collision mesh filename=package://bit_humanoid/meshes/ranklepitch.STL; visual mesh filename=package://bit_humanoid/meshes/ranklepitch.STL
- link rankleroll: geometry collision mesh filename=package://bit_humanoid/meshes/rankleroll.STL; visual mesh filename=package://bit_humanoid/meshes/rankleroll.STL
- link rhippitch: geometry collision mesh filename=package://bit_humanoid/meshes/rhippitch.STL; visual mesh filename=package://bit_humanoid/meshes/rhippitch.STL
- link rhiproll: geometry collision mesh filename=package://bit_humanoid/meshes/rhiproll.STL; visual mesh filename=package://bit_humanoid/meshes/rhiproll.STL
- link rhipyaw: geometry collision mesh filename=package://bit_humanoid/meshes/rhipyaw.STL; visual mesh filename=package://bit_humanoid/meshes/rhipyaw.STL
- link rkneepitch: geometry collision mesh filename=package://bit_humanoid/meshes/rkneepitch.STL; visual mesh filename=package://bit_humanoid/meshes/rkneepitch.STL
- link torso: geometry collision mesh filename=package://bit_humanoid/meshes/torso.STL; visual mesh filename=package://bit_humanoid/meshes/torso.STL
